File: ButterflyChain.kicad_pcb (KiCad board)
At the start: 2 copper layers, 93.1 x 65.5 mm, 26 parts, among them J1 Input, J2 Output, J3 Antennae

Commit message: Label LEDs on silkscreen.  (0-based numbering)
Other:
- board text added: "0"
- board text added: "1"
- board text added: "10"
- board text added: "11"
- board text added: "12"
- board text added: "13"
- board text added: "14"
- board text added: "15"
- board text added: "16"
- board text added: "17"
- board text added: "2"
- board text added: "3"
- board text added: "4"
- board text added: "5"
- board text added: "6"
- board text added: "7"
- board text added: "8"
- board text added: "9"
Changed lines of the file:
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@@
     (area 53.34 73.047739 147.320001 139.700001)
     (thickness 1.6)
-    (drawings 191)
+    (drawings 209)
     (tracks 250)
     (zones 0)
@@
   (title_block
     (title "Chainable NeoPixel Butterfly")
-    (date 2018-09-02)
+    (date 2018-09-03)
     (rev 1.0)
     (company "Patrick Pelletier")
@@
     (36 B.SilkS user)
     (37 F.SilkS user)
-    (38 B.Mask user hide)
+    (38 B.Mask user)
     (39 F.Mask user)
     (40 Dwgs.User user)
@@
     (pad_to_mask_clearance 0)
     (aux_axis_origin 0 0)
-    (visible_elements FFFEF77F)
+    (visible_elements FFFEF7FF)
     (pcbplotparams
       (layerselection 0x010f0_80000001)
@@
       (xy 0.286924 -3.969467) (xy 0.724974 -3.940798)) (layer F.SilkS) (width 0.01))
   )
+  (gr_text 17 (at 83 119.5) (layer B.SilkS)
+    (effects (font (size 1.5 1.5) (thickness 0.3)) (justify mirror))
+  )
+  (gr_text 16 (at 74 124.5) (layer B.SilkS)
+    (effects (font (size 1.5 1.5) (thickness 0.3)) (justify mirror))
+  )
+  (gr_text 15 (at 78 109.5) (layer B.SilkS)
+    (effects (font (size 1.5 1.5) (thickness 0.3)) (justify mirror))
+  )
+  (gr_text 14 (at 62 92.5) (layer B.SilkS)
+    (effects (font (size 1.5 1.5) (thickness 0.3)) (justify mirror))
+  )
+  (gr_text 13 (at 74 99.5) (layer B.SilkS)
+    (effects (font (size 1.5 1.5) (thickness 0.3)) (justify mirror))
+  )
+  (gr_text 12 (at 86 104.5) (layer B.SilkS)
+    (effects (font (size 1.5 1.5) (thickness 0.3)) (justify mirror))
+  )
+  (gr_text 11 (at 61 79.5) (layer B.SilkS)
+    (effects (font (size 1.5 1.5) (thickness 0.3)) (justify mirror))
+  )
+  (gr_text 10 (at 72.5 88.5) (layer B.SilkS)
+    (effects (font (size 1.5 1.5) (thickness 0.3)) (justify mirror))
+  )
+  (gr_text 9 (at 85 95.5) (layer B.SilkS)
+    (effects (font (size 1.5 1.5) (thickness 0.3)) (justify mirror))
+  )
+  (gr_text 8 (at 117.5 119.5) (layer B.SilkS)
+    (effects (font (size 1.5 1.5) (thickness 0.3)) (justify mirror))
+  )
+  (gr_text 7 (at 126.5 124.5) (layer B.SilkS)
+    (effects (font (size 1.5 1.5) (thickness 0.3)) (justify mirror))
+  )
+  (gr_text 6 (at 122.5 109.5) (layer B.SilkS)
+    (effects (font (size 1.5 1.5) (thickness 0.3)) (justify mirror))
+  )
+  (gr_text 5 (at 138.5 92.5) (layer B.SilkS)
+    (effects (font (size 1.5 1.5) (thickness 0.3)) (justify mirror))
+  )
+  (gr_text 4 (at 126.5 99.5) (layer B.SilkS)
+    (effects (font (size 1.5 1.5) (thickness 0.3)) (justify mirror))
+  )
+  (gr_text 3 (at 114.5 104.5) (layer B.SilkS)
+    (effects (font (size 1.5 1.5) (thickness 0.3)) (justify mirror))
+  )
+  (gr_text 2 (at 139.5 79.5) (layer B.SilkS)
+    (effects (font (size 1.5 1.5) (thickness 0.3)) (justify mirror))
+  )
+  (gr_text 1 (at 127.5 88.5) (layer B.SilkS)
+    (effects (font (size 1.5 1.5) (thickness 0.3)) (justify mirror))
+  )
+  (gr_text 0 (at 115.5 95.5) (layer B.SilkS)
+    (effects (font (size 1.5 1.5) (thickness 0.3)) (justify mirror))
+  )
   (gr_text GND (at 123.5 111.5) (layer F.SilkS)

Commit message: Add text "Butterfly!" to silkscreen.
Other:
- board text added: "Butterfly!"
Changed lines of the file:
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@@
     (area 53.34 73.047739 147.320001 139.700001)
     (thickness 1.6)
-    (drawings 209)
+    (drawings 210)
     (tracks 250)
     (zones 0)
@@
       (xy 0.286924 -3.969467) (xy 0.724974 -3.940798)) (layer F.SilkS) (width 0.01))
   )
+  (gr_text Butterfly! (at 100 106 90) (layer B.SilkS)
+    (effects (font (size 2.5 2.5) (thickness 0.5)) (justify mirror))
+  )
   (gr_text 17 (at 83 119.5) (layer B.SilkS)
